Commit message: [ur_common][urdf] added D405 placeholder and attached robotiq FT sensor and 2f-85 gripper to the ur_common urdf

File: ur_description/urdf/inc/ur_macro.xacro (robot description, xacro)
@@ -206,4 +206,26 @@
       </xacro:cylinder_inertial>
     </link>
+    <!-- white material for camera -->
+    <material name="white">
+      <color rgba="1 1 1 1"/>
+    </material>
+    <!-- Placeholder box for D405 camera -->
+    <link name="${prefix}camera_link">
+      <inertial>
+        <mass value="1.0" />
+        <inertia  ixx="1.0" ixy="0.0"  ixz="0.0"  iyy="100.0"  iyz="0.0"  izz="1.0" />
+      </inertial>
+      <visual>
+        <geometry>
+          <box size="0.025 0.045 0.045" />
+        </geometry>
+        <material name="white"/>
+      </visual>
+      <collision>
+        <geometry>
+          <box size="0.025 0.045 0.045" />
+        </geometry>
+      </collision>
+    </link>
     <!-- joints: main serial chain -->
     <joint name="${prefix}base_link-base_link_inertia" type="fixed">
@@ -301,5 +323,5 @@
       <child link="${prefix}base"/>
     </joint>
-    <!-- ROS-Industrial 'flange' frame: attachment point for EEF models -->
+    <!-- ROS-Industrial 'flange' frame attachment point for EEF models -->
     <link name="${prefix}flange" />
     <joint name="${prefix}wrist_3-flange" type="fixed">
@@ -316,4 +338,23 @@
       <child link="${prefix}tool0"/>
     </joint>
+    <!-- D405 Camera -->
+    <joint name="camera" type="fixed">
+      <origin xyz="0.0 0.05 0.0575" rpy="-${pi/2} -${pi/2} 0"/>
+      <parent link="${prefix}wrist_3_link"/>
+      <child link="${prefix}camera_link"/>
+    </joint>
+    <!-- FT sensor -->
+    <xacro:include filename="$(find robotiq_ft_sensor)/urdf/robotiq_ft300.urdf.xacro" />
+    <xacro:robotiq_ft300 prefix="${prefix}ft_" parent="${prefix}wrist_3_link">
+      <origin xyz="0 0 -0.005" rpy="0 0 0" />
+    </xacro:robotiq_ft300>
+    <!-- Robotiq 2f-85 gripper -->
+    <xacro:include filename="$(find robotiq_2f_85_gripper_visualization)/urdf/robotiq_arg2f_85_model_macro.xacro" />
+    <xacro:robotiq_arg2f_85 prefix="${prefix}gripper_" />
+    <joint name="${prefix}gripper_joint" type="fixed">
+      <parent link="${prefix}ft_ft300_sensor" />
+      <child link="${prefix}gripper_robotiq_arg2f_base_link"/>
+      <origin xyz="0 0 0.01" rpy="0 ${pi} ${-pi/2}"/>
+    </joint>
   </xacro:macro>
 </robot>

Commit message: [urdf][moveit_config] added grasp point to the urdf and shelf_pick home pose to srdf

File: ur_description/urdf/inc/ur_macro.xacro (robot description, xacro)
@@ -357,4 +357,18 @@
       <origin xyz="0 0 0.01" rpy="0 ${pi} ${-pi/2}"/>
     </joint>
+    <!-- Virtual Grasp Point Link -->
+    <link name="${prefix}2f_85_grasp_point">
+    </link>
+    <!-- Virtual Grasp Point Fixed Joint -->
+    <joint name="${prefix}2f_85_grasp_point_joint" type="fixed">
+        <parent link="${prefix}gripper_robotiq_arg2f_base_link"/>
+        <child link="${prefix}2f_85_grasp_point"/>
+        <!-- Center between finger tips -->
+        <!-- RPY - Matching the convention (same as tool0)-->
+        <!-- Z Offset - gripper length closed minus half the finger pads -->
+        <!-- <origin rpy="0 0 -1.570796325" xyz="0 0 ${0.1628-0.038/2}"/> -->
+        <!-- Z Offset - gripper length closed -->
+        <origin rpy="0 0 -1.570796325" xyz="0 0 0.1628"/>
+    </joint>
   </xacro:macro>
 </robot>

Commit message: [urdf] added gripper coupler and table to the urdf

File: ur_description/urdf/inc/ur_macro.xacro (robot description, xacro)
@@ -63,4 +63,22 @@
     <!-- Add URDF transmission elements (for ros_control) -->
     <xacro:ur_arm_transmission prefix="${prefix}" hw_interface="${transmission_hw_interface}" />
+    <!-- links -->
+    <link name="${prefix}table">
+      <visual>
+        <origin rpy="0 0 ${pi/2}" xyz="-0.225 0.415 -0.45"/>
+        <geometry>
+          <box size="1.00 0.80 0.90"/>
+        </geometry>
+        <material name="white">
+          <color rgba="1 1 1 1"/>
+        </material>
+      </visual>
+      <collision>
+        <origin rpy="0 0 ${pi/2}" xyz="-0.225 0.415 -0.45"/>
+        <geometry>
+          <box size="1.00 0.80 0.90"/>
+        </geometry>
+      </collision>
+    </link>
     <!-- links: main serial chain -->
     <link name="${prefix}base_link"/>
@@ -85,4 +103,9 @@
       </xacro:cylinder_inertial>
     </link>
+    <joint name="${prefix}table_to_base_link" type="fixed">
+      <parent link="${prefix}table"/>
+      <child link="${prefix}base_link"/>
+      <origin xyz="0 0 0" rpy="0 0 0"/>
+    </joint>
     <link name="${prefix}shoulder_link">
       <visual>
@@ -205,26 +228,4 @@
         <origin xyz="0.0 0.0 ${-0.5 * wrist_3_inertia_length}" rpy="0 0 0" />
       </xacro:cylinder_inertial>
-    </link>
-    <!-- white material for camera -->
-    <material name="white">
-      <color rgba="1 1 1 1"/>
-    </material>
-    <!-- Placeholder box for D405 camera -->
-    <link name="${prefix}camera_link">
-      <inertial>
-        <mass value="1.0" />
-        <inertia  ixx="1.0" ixy="0.0"  ixz="0.0"  iyy="100.0"  iyz="0.0"  izz="1.0" />
-      </inertial>
-      <visual>
-        <geometry>
-          <box size="0.025 0.045 0.045" />
-        </geometry>
-        <material name="white"/>
-      </visual>
-      <collision>
-        <geometry>
-          <box size="0.025 0.045 0.045" />
-        </geometry>
-      </collision>
     </link>
     <!-- joints: main serial chain -->
@@ -338,22 +339,63 @@
       <child link="${prefix}tool0"/>
     </joint>
+    <!-- Placeholder box for D405 camera -->
+    <link name="${prefix}camera_link">
+      <inertial>
+        <mass value="1.0" />
+        <inertia  ixx="1.0" ixy="0.0"  ixz="0.0"  iyy="100.0"  iyz="0.0"  izz="1.0" />
+      </inertial>
+      <visual>
+        <geometry>
+          <box size="0.025 0.045 0.045" />
+        </geometry>
+        <material name="white">
+          <color rgba="1 1 1 1"/>
+        </material>
+      </visual>
+      <collision>
+        <geometry>
+          <box size="0.025 0.045 0.045" />
+        </geometry>
+      </collision>
+    </link>
     <!-- D405 Camera -->
     <joint name="camera" type="fixed">
-      <origin xyz="0.0 0.05 0.0575" rpy="-${pi/2} -${pi/2} 0"/>
+      <origin xyz="0.0 0.065 0.035" rpy="-${pi/2} -${pi/2} 0"/>
       <parent link="${prefix}wrist_3_link"/>
       <child link="${prefix}camera_link"/>
     </joint>
-    <!-- FT sensor -->
-    <xacro:include filename="$(find robotiq_ft_sensor)/urdf/robotiq_ft300.urdf.xacro" />
-    <xacro:robotiq_ft300 prefix="${prefix}ft_" parent="${prefix}wrist_3_link">
-      <origin xyz="0 0 -0.005" rpy="0 0 0" />
-    </xacro:robotiq_ft300>
+    <link name="${prefix}robotiq_coupler">
+      <visual>
+        <geometry>
+          <mesh filename="package://robotiq_2f_85_gripper_visualization/meshes/robotiq_85_coupler.stl" />
+        </geometry>
+        <material name="">
+            <color rgba="0.1 0.1 0.1 1"/>
+        </material>
+      </visual>
+      <collision>
+        <geometry>
+          <mesh filename="package://robotiq_2f_85_gripper_visualization/meshes/robotiq_85_coupler.stl" />
+        </geometry>
+      </collision>
+      <inertial>
+        <origin xyz="2.073e-05   1.45286e-03  -1.1049e-03" rpy="0 0 0" />
+        <mass value="0.168" />
+        <inertia ixx="6.69695624e-05" ixy="5.21511788e-09" ixz="-2.74383009e-08"
+                iyy="7.85088161e-05" iyz="5.41105193e-07" izz="1.41819717e-04"/>
+      </inertial>
+    </link>
+    <joint name="${prefix}robotiq_coupler_joint" type="fixed">
+      <origin xyz="0 0 0.004" rpy="0 0 0" />
+      <parent link="${prefix}tool0"/>
+      <child link="${prefix}robotiq_coupler"/>
+    </joint>
     <!-- Robotiq 2f-85 gripper -->
     <xacro:include filename="$(find robotiq_2f_85_gripper_visualization)/urdf/robotiq_arg2f_85_model_macro.xacro" />
     <xacro:robotiq_arg2f_85 prefix="${prefix}gripper_" />
     <joint name="${prefix}gripper_joint" type="fixed">
-      <parent link="${prefix}ft_ft300_sensor" />
+      <parent link="${prefix}robotiq_coupler" />
       <child link="${prefix}gripper_robotiq_arg2f_base_link"/>
-      <origin xyz="0 0 0.01" rpy="0 ${pi} ${-pi/2}"/>
+      <origin xyz="0 0 0.005" rpy="${pi} ${pi} ${-pi/2}"/>
     </joint>
     <!-- Virtual Grasp Point Link -->
@@ -364,10 +406,5 @@
         <parent link="${prefix}gripper_robotiq_arg2f_base_link"/>
         <child link="${prefix}2f_85_grasp_point"/>
-        <!-- Center between finger tips -->
-        <!-- RPY - Matching the convention (same as tool0)-->
-        <!-- Z Offset - gripper length closed minus half the finger pads -->
-        <!-- <origin rpy="0 0 -1.570796325" xyz="0 0 ${0.1628-0.038/2}"/> -->
-        <!-- Z Offset - gripper length closed -->
-        <origin rpy="0 0 -1.570796325" xyz="0 0 0.1628"/>
+        <origin rpy="${pi} -${pi/2} 0" xyz="0 0 0.1628"/>
     </joint>
   </xacro:macro>

Commit message: [urdf] added gripper coupler mesh file

File: ur_description/urdf/inc/ur_macro.xacro (robot description, xacro)
@@ -368,5 +368,5 @@
       <visual>
         <geometry>
-          <mesh filename="package://robotiq_2f_85_gripper_visualization/meshes/robotiq_85_coupler.stl" />
+          <mesh filename="package://ur_description/meshes/ur5/robotiq_85_coupler.stl" />
         </geometry>
         <material name="">
@@ -376,5 +376,5 @@
       <collision>
         <geometry>
-          <mesh filename="package://robotiq_2f_85_gripper_visualization/meshes/robotiq_85_coupler.stl" />
+          <mesh filename="package://ur_description/meshes/ur5/meshes/robotiq_85_coupler.stl" />
         </geometry>
       </collision>

Commit message: [urdf] added second camera along with its stand

File: ur_description/urdf/inc/ur_macro.xacro (robot description, xacro)
@@ -376,5 +376,5 @@
       <collision>
         <geometry>
-          <mesh filename="package://ur_description/meshes/ur5/meshes/robotiq_85_coupler.stl" />
+          <mesh filename="package://ur_description/meshes/ur5/robotiq_85_coupler.stl" />
         </geometry>
       </collision>
@@ -408,4 +408,166 @@
         <origin rpy="${pi} -${pi/2} 0" xyz="0 0 0.1628"/>
     </joint>
+    <!-- wall -->
+    <link name="${prefix}wall">
+      <visual>
+        <geometry>
+          <box size="0.01 2.5 3.0" />
+        </geometry>
+        <material name="">
+            <color rgba="1 0.9 0.7 1"/>
+        </material>
+      </visual>
+      <collision>
+        <geometry>
+          <box size="0.01 2.5 3.0" />
+        </geometry>
+      </collision>
+      <inertial>
+        <origin xyz="0 0 0" rpy="0 0 0" />
+        <mass value="1" />
+        <inertia ixx="1" ixy="0" ixz="0"
+                iyy="1" iyz="0" izz="1"/>
+      </inertial>
+    </link>
+    <joint name="${prefix}wall_joint" type="fixed">
+      <origin xyz="0.665 0.0 0" rpy="0 0 0" />
+      <parent link="${prefix}base"/>
+      <child link="${prefix}wall"/>
+    </joint>
+    <!-- camera stand -->
+    <link name="${prefix}camera_stand">
+      <visual>
+        <geometry>
+          <box size="0.02 0.04 0.76" />
+        </geometry>
+        <material name="">
+            <color rgba="0.85098 0.85098 0.85098 1"/>
+        </material>
+      </visual>
+      <collision>
+        <geometry>
+          <box size="0.02 0.04 0.76" />
+        </geometry>
+      </collision>
+      <inertial>
+        <origin xyz="0 0 0" rpy="0 0 0" />
+        <mass value="1" />
+        <inertia ixx="1" ixy="0" ixz="0"
+                iyy="1" iyz="0" izz="1"/>
+      </inertial>
+    </link>
+    <joint name="${prefix}camera_stand_joint" type="fixed">
+      <origin xyz="0.645 -0.415 0.38" rpy="0 0 0" />
+      <parent link="${prefix}base"/>
+      <child link="${prefix}camera_stand"/>
+    </joint>
+    <!-- camera stand horizontal -->
+    <link name="${prefix}camera_stand_horizontal">
+      <visual>
+        <geometry>
+          <box size="0.02 0.72 0.02" />
+        </geometry>
+        <material name="">
+            <color rgba="0.85098 0.85098 0.85098 1"/>
+        </material>
+      </visual>
+      <collision>
+        <geometry>
+          <box size="0.02 0.76 0.02" />
+        </geometry>
+      </collision>
+      <inertial>
+        <origin xyz="0 0 0" rpy="0 0 0" />
+        <mass value="1" />
+        <inertia ixx="1" ixy="0" ixz="0"
+                iyy="1" iyz="0" izz="1"/>
+      </inertial>
+    </link>
+    <joint name="${prefix}camera_stand_horizontal_joint" type="fixed">
+      <origin xyz="-0.36 0.0 0.38" rpy="0 0 ${pi/2}" />
+      <parent link="${prefix}camera_stand"/>
+      <child link="${prefix}camera_stand_horizontal"/>
+    </joint>
+    <!-- camera stand horizontal -->
+    <link name="${prefix}camera_stand_horizontal2">
+      <visual>
+        <geometry>
+          <box size="0.02 0.53 0.02" />
+        </geometry>
+        <material name="">
+            <color rgba="0.85098 0.85098 0.85098 1"/>
+        </material>
+      </visual>
+      <collision>
+        <geometry>
+          <box size="0.02 0.53 0.02" />
+        </geometry>
+      </collision>
+      <inertial>
+        <origin xyz="0 0 0" rpy="0 0 0" />
+        <mass value="1" />
+        <inertia ixx="1" ixy="0" ixz="0"
+                iyy="1" iyz="0" izz="1"/>
+      </inertial>
+    </link>
+    <joint name="${prefix}camera_stand_horizontal_joint2" type="fixed">
+      <origin xyz="0.0 0.0 0.0" rpy="0 0 0" />
+      <parent link="${prefix}camera_stand_horizontal"/>
+      <child link="${prefix}camera_stand_horizontal2"/>
+    </joint>
+    <!-- camera ring -->
+    <link name="${prefix}camera_ring">
+      <visual>
+        <geometry>
+          <cylinder length="0.02" radius="0.24" />
+        </geometry>
+        <material name="">
+            <color rgba="0.85098 0.85098 0.85098 1"/>
+        </material>
+      </visual>
+      <collision>
+        <geometry>
+          <cylinder length="0.04" radius="0.24" />
+        </geometry>
+      </collision>
+      <inertial>
+        <origin xyz="0 0 0" rpy="0 0 0" />
+        <mass value="1" />
+        <inertia ixx="1" ixy="0" ixz="0"
+                iyy="1" iyz="0" izz="1"/>
+      </inertial>
+    </link>
+    <joint name="${prefix}camera_ring_joint" type="fixed">
+      <origin xyz="0.0 0.0 -0.4" rpy="0 0 0" />
+      <parent link="${prefix}camera_stand_horizontal2"/>
+      <child link="${prefix}camera_ring"/>
+    </joint>
+    <!-- camera -->
+    <link name="${prefix}camera2">
+      <visual>
+        <geometry>
+          <cylinder length="0.04" radius="0.24" />
+        </geometry>
+        <material name="">
+            <color rgba="0.85098 0.85098 0.85098 1"/>
+        </material>
+      </visual>
+      <collision>
+        <geometry>
+          <cylinder length="0.04" radius="0.24" />
+        </geometry>
+      </collision>
+      <inertial>
+        <origin xyz="0 0 0" rpy="0 0 0" />
+        <mass value="1" />
+        <inertia ixx="1" ixy="0" ixz="0"
+                iyy="1" iyz="0" izz="1"/>
+      </inertial>
+    </link>
+    <joint name="${prefix}camera2_joint" type="fixed">
+      <origin xyz="0.0 0.0 -0.4" rpy="0 0 0" />
+      <parent link="${prefix}camera_ring"/>
+      <child link="${prefix}camera2"/>
+    </joint>
   </xacro:macro>
 </robot>

Commit message: [urdf] modified the urdf to add second camera setup

File: ur_description/urdf/inc/ur_macro.xacro (robot description, xacro)
@@ -466,5 +466,5 @@
       <visual>
         <geometry>
-          <box size="0.02 0.72 0.02" />
+          <box size="0.025 0.72 0.025" />
         </geometry>
         <material name="">
@@ -474,5 +474,5 @@
       <collision>
         <geometry>
-          <box size="0.02 0.76 0.02" />
+          <box size="0.025 0.76 0.025" />
         </geometry>
       </collision>
@@ -493,5 +493,5 @@
       <visual>
         <geometry>
-          <box size="0.02 0.53 0.02" />
+          <box size="0.025 0.53 0.025" />
         </geometry>
         <material name="">
@@ -501,5 +501,5 @@
       <collision>
         <geometry>
-          <box size="0.02 0.53 0.02" />
+          <box size="0.025 0.53 0.025" />
         </geometry>
       </collision>
@@ -512,5 +512,5 @@
     </link>
     <joint name="${prefix}camera_stand_horizontal_joint2" type="fixed">
-      <origin xyz="0.0 0.0 0.0" rpy="0 0 0" />
+      <origin xyz="0.0 0.0 0.0" rpy="0 0 ${pi/2}" />
       <parent link="${prefix}camera_stand_horizontal"/>
       <child link="${prefix}camera_stand_horizontal2"/>
@@ -528,5 +528,5 @@
       <collision>
         <geometry>
-          <cylinder length="0.04" radius="0.24" />
+          <cylinder length="0.02" radius="0.24" />
         </geometry>
       </collision>
@@ -539,5 +539,5 @@
     </link>
     <joint name="${prefix}camera_ring_joint" type="fixed">
-      <origin xyz="0.0 0.0 -0.4" rpy="0 0 0" />
+      <origin xyz="0.0 0.0 -0.025" rpy="0 0 0" />
       <parent link="${prefix}camera_stand_horizontal2"/>
       <child link="${prefix}camera_ring"/>
@@ -547,13 +547,13 @@
       <visual>
         <geometry>
-          <cylinder length="0.04" radius="0.24" />
-        </geometry>
-        <material name="">
-            <color rgba="0.85098 0.85098 0.85098 1"/>
-        </material>
-      </visual>
-      <collision>
-        <geometry>
-          <cylinder length="0.04" radius="0.24" />
+          <cylinder length="0.03" radius="0.03" />
+        </geometry>
+        <material name="white">
+          <color rgba="1 1 1 1"/>
+        </material>
+      </visual>
+      <collision>
+        <geometry>
+          <cylinder length="0.03" radius="0.03" />
         </geometry>
       </collision>
@@ -566,5 +566,5 @@
     </link>
     <joint name="${prefix}camera2_joint" type="fixed">
-      <origin xyz="0.0 0.0 -0.4" rpy="0 0 0" />
+      <origin xyz="0.0 0.0 -0.015" rpy="0 0 0" />
       <parent link="${prefix}camera_ring"/>
       <child link="${prefix}camera2"/>

Commit message: [urdf] increased hand-cam collision limits

File: ur_description/urdf/inc/ur_macro.xacro (robot description, xacro)
@@ -355,5 +355,5 @@
       <collision>
         <geometry>
-          <box size="0.025 0.045 0.045" />
+          <box size="0.055 0.075 0.075" />
         </geometry>
       </collision>
