Commit message: [ma_scvp] configured urdf and moveit for ma_scvp_real setup

File: ur_description/urdf/inc/ur_macro.xacro (robot description, xacro)
@@ -339,6 +339,6 @@
       <child link="${prefix}tool0"/>
     </joint>
-    <!-- Placeholder box for D405 camera -->
-    <link name="${prefix}camera_link">
+    <!-- camera mount -->
+    <link name="${prefix}camera_mount_link">
       <inertial>
         <mass value="1.0" />
@@ -347,5 +347,5 @@
       <visual>
         <geometry>
-          <box size="0.025 0.045 0.045" />
+          <box size="0.015 0.015 0.035" />
         </geometry>
         <material name="white">
@@ -355,57 +355,18 @@
       <collision>
         <geometry>
-          <box size="0.055 0.075 0.075" />
-        </geometry>
-      </collision>
-    </link>
-    <!-- D405 Camera -->
-    <joint name="camera" type="fixed">
-      <origin xyz="0.0 0.065 0.035" rpy="-${pi/2} -${pi/2} 0"/>
-      <parent link="${prefix}wrist_3_link"/>
-      <child link="${prefix}camera_link"/>
-    </joint>
-    <link name="${prefix}robotiq_coupler">
-      <visual>
-        <geometry>
-          <mesh filename="package://ur_description/meshes/ur5/robotiq_85_coupler.stl" />
-        </geometry>
-        <material name="">
-            <color rgba="0.1 0.1 0.1 1"/>
-        </material>
-      </visual>
-      <collision>
-        <geometry>
-          <mesh filename="package://ur_description/meshes/ur5/robotiq_85_coupler.stl" />
-        </geometry>
-      </collision>
-      <inertial>
-        <origin xyz="2.073e-05   1.45286e-03  -1.1049e-03" rpy="0 0 0" />
-        <mass value="0.168" />
-        <inertia ixx="6.69695624e-05" ixy="5.21511788e-09" ixz="-2.74383009e-08"
-                iyy="7.85088161e-05" iyz="5.41105193e-07" izz="1.41819717e-04"/>
-      </inertial>
-    </link>
-    <joint name="${prefix}robotiq_coupler_joint" type="fixed">
-      <origin xyz="0 0 0.004" rpy="0 0 0" />
-      <parent link="${prefix}tool0"/>
-      <child link="${prefix}robotiq_coupler"/>
-    </joint>
-    <!-- Robotiq 2f-85 gripper -->
-    <xacro:include filename="$(find robotiq_2f_85_gripper_visualization)/urdf/robotiq_arg2f_85_model_macro.xacro" />
-    <xacro:robotiq_arg2f_85 prefix="${prefix}gripper_" />
-    <joint name="${prefix}gripper_joint" type="fixed">
-      <parent link="${prefix}robotiq_coupler" />
-      <child link="${prefix}gripper_robotiq_arg2f_base_link"/>
-      <origin xyz="0 0 0.005" rpy="${pi} ${pi} ${-pi/2}"/>
-    </joint>
-    <!-- Virtual Grasp Point Link -->
-    <link name="${prefix}2f_85_grasp_point">
-    </link>
-    <!-- Virtual Grasp Point Fixed Joint -->
-    <joint name="${prefix}2f_85_grasp_point_joint" type="fixed">
-        <parent link="${prefix}gripper_robotiq_arg2f_base_link"/>
-        <child link="${prefix}2f_85_grasp_point"/>
-        <origin rpy="${pi} -${pi/2} 0" xyz="0 0 0.1628"/>
-    </joint>
+          <box size="0.015 0.015 0.035" />
+        </geometry>
+      </collision>
+    </link>
+    <joint name="camera_mount" type="fixed">
+      <origin xyz="0.0 0.0 0.0175" rpy="0.0 0.0 0.0" />
+      <parent link="${prefix}wrist_3_link" />
+      <child link="${prefix}camera_mount_link" />
+    </joint>
+    <!-- include realsense d435 camera -->
+    <xacro:include filename="$(find realsense2_description)/urdf/_d435.urdf.xacro" />
+    <xacro:sensor_d435 name="camera" parent="${prefix}camera_mount_link">
+      <origin xyz="-0.013 0.0 0.0275" rpy="${pi} -${pi/2} 0.0" />
+    </xacro:sensor_d435>
     <!-- wall -->
     <link name="${prefix}wall">
@@ -462,112 +423,4 @@
       <child link="${prefix}camera_stand"/>
     </joint>
-    <!-- camera stand horizontal -->
-    <link name="${prefix}camera_stand_horizontal">
-      <visual>
-        <geometry>
-          <box size="0.025 0.72 0.025" />
-        </geometry>
-        <material name="">
-            <color rgba="0.85098 0.85098 0.85098 1"/>
-        </material>
-      </visual>
-      <collision>
-        <geometry>
-          <box size="0.025 0.76 0.025" />
-        </geometry>
-      </collision>
-      <inertial>
-        <origin xyz="0 0 0" rpy="0 0 0" />
-        <mass value="1" />
-        <inertia ixx="1" ixy="0" ixz="0"
-                iyy="1" iyz="0" izz="1"/>
-      </inertial>
-    </link>
-    <joint name="${prefix}camera_stand_horizontal_joint" type="fixed">
-      <origin xyz="-0.36 0.0 0.38" rpy="0 0 ${pi/2}" />
-      <parent link="${prefix}camera_stand"/>
-      <child link="${prefix}camera_stand_horizontal"/>
-    </joint>
-    <!-- camera stand horizontal -->
-    <link name="${prefix}camera_stand_horizontal2">
-      <visual>
-        <geometry>
-          <box size="0.025 0.53 0.025" />
-        </geometry>
-        <material name="">
-            <color rgba="0.85098 0.85098 0.85098 1"/>
-        </material>
-      </visual>
-      <collision>
-        <geometry>
-          <box size="0.025 0.53 0.025" />
-        </geometry>
-      </collision>
-      <inertial>
-        <origin xyz="0 0 0" rpy="0 0 0" />
-        <mass value="1" />
-        <inertia ixx="1" ixy="0" ixz="0"
-                iyy="1" iyz="0" izz="1"/>
-      </inertial>
-    </link>
-    <joint name="${prefix}camera_stand_horizontal_joint2" type="fixed">
-      <origin xyz="0.0 0.0 0.0" rpy="0 0 ${pi/2}" />
-      <parent link="${prefix}camera_stand_horizontal"/>
-      <child link="${prefix}camera_stand_horizontal2"/>
-    </joint>
-    <!-- camera ring -->
-    <link name="${prefix}camera_ring">
-      <visual>
-        <geometry>
-          <cylinder length="0.02" radius="0.24" />
-        </geometry>
-        <material name="">
-            <color rgba="0.85098 0.85098 0.85098 1"/>
-        </material>
-      </visual>
-      <collision>
-        <geometry>
-          <cylinder length="0.02" radius="0.24" />
-        </geometry>
-      </collision>
-      <inertial>
-        <origin xyz="0 0 0" rpy="0 0 0" />
-        <mass value="1" />
-        <inertia ixx="1" ixy="0" ixz="0"
-                iyy="1" iyz="0" izz="1"/>
-      </inertial>
-    </link>
-    <joint name="${prefix}camera_ring_joint" type="fixed">
-      <origin xyz="0.0 0.0 -0.025" rpy="0 0 0" />
-      <parent link="${prefix}camera_stand_horizontal2"/>
-      <child link="${prefix}camera_ring"/>
-    </joint>
-    <!-- camera -->
-    <link name="${prefix}camera2">
-      <visual>
-        <geometry>
-          <cylinder length="0.03" radius="0.03" />
-        </geometry>
-        <material name="white">
-          <color rgba="1 1 1 1"/>
-        </material>
-      </visual>
-      <collision>
-        <geometry>
-          <cylinder length="0.03" radius="0.03" />
-        </geometry>
-      </collision>
-      <inertial>
-        <origin xyz="0 0 0" rpy="0 0 0" />
-        <mass value="1" />
-        <inertia ixx="1" ixy="0" ixz="0"
-                iyy="1" iyz="0" izz="1"/>
-      </inertial>
-    </link>
-    <joint name="${prefix}camera2_joint" type="fixed">
-      <origin xyz="0.0 0.0 -0.015" rpy="0 0 0" />
-      <parent link="${prefix}camera_ring"/>
-      <child link="${prefix}camera2"/>
-    </joint>
   </xacro:macro>
 </robot>

Commit message: [urdf] updated d435 position

File: ur_description/urdf/inc/ur_macro.xacro (robot description, xacro)
@@ -364,8 +364,34 @@
       <child link="${prefix}camera_mount_link" />
     </joint>
+    <!-- <link name="${prefix}camera_link">
+      <inertial>
+        <mass value="1.0" />
+        <inertia  ixx="1.0" ixy="0.0"  ixz="0.0"  iyy="100.0"  iyz="0.0"  izz="1.0" />
+      </inertial>
+      <visual>
+        <geometry>
+          <box size="0.025 0.045 0.045" />
+        </geometry>
+        <material name="white">
+          <color rgba="1 1 1 1"/>
+        </material>
+      </visual>
+      <collision>
+        <geometry>
+          <box size="0.055 0.075 0.075" />
+        </geometry>
+      </collision>
+    </link>
+    <joint name="camera" type="fixed">
+      <origin xyz="-0.000614899 0.0332126 0.0588194" rpy="${0.00391367/pi} ${0.00134805/pi} ${1.56867/pi}" />
+      <parent link="${prefix}wrist_3_link"/>
+      <child link="${prefix}camera_link"/>
+    </joint> -->
     <!-- include realsense d435 camera -->
     <xacro:include filename="$(find realsense2_description)/urdf/_d435.urdf.xacro" />
     <xacro:sensor_d435 name="camera" parent="${prefix}camera_mount_link">
-      <origin xyz="-0.013 0.0 0.0275" rpy="${pi} -${pi/2} 0.0" />
+      <!-- <origin xyz="-0.013 0.0 0.0275" rpy="${pi} -${pi/2} 0.0" /> -->
+      <!-- <origin xyz="0.000614899 -0.0332126 0.0588194" rpy="0.00391367 0.00134805 1.56867" /> -->
+      <origin xyz="-0.013 0.0 0.0275" rpy="${-pi / 2} ${-pi / 2} ${-pi / 2}" />
     </xacro:sensor_d435>
     <!-- wall -->
